Commit message: the automated person model is now complete

File: bwi_gazebo_entities/gazebo/automated_person.gazebo.xacro (robot description, xacro)
@@ -19,5 +19,5 @@
         <updateRate>${update_rate}</updateRate>
         <controller:gazebo_ros_laser name="gazebo_ros_${name}_controller" plugin="libgazebo_ros_laser.so">
-          <gaussianNoise>0.03</gaussianNoise>
+          <gaussianNoise>0</gaussianNoise>
           <alwaysOn>true</alwaysOn>
           <updateRate>${update_rate}</updateRate>

File: bwi_gazebo_entities/urdf/person.urdf.xacro (robot description, xacro)
@@ -1,4 +1,5 @@
 <?xml version="1.0"?>
 <root xmlns:xacro="http://ros.org/wiki/xacro">
+  <include filename="$(find bwi_gazebo_entities)/urdf/person.gazebo.xacro" />
   <xacro:macro name="person">
     <!-- root link, on the ground just below the person origin (torso) -->
@@ -12,5 +13,5 @@
     </link>
     <joint name="base_link_joint" type="fixed">
-      <origin xyz="0.0 0 1.25" rpy="0 0 0" />
+      <origin xyz="0.0 0 1.0" rpy="0 0 0" />
       <parent link="base_footprint"/>
       <child link="base_link" />
@@ -19,5 +20,5 @@
     <link name="base_link">
       <inertial>
-        <mass value="40" />
+        <mass value="0.01" />
         <origin xyz="0 0 0" />
         <inertia ixx="1.0" ixy="0.0" ixz="0.0"
@@ -27,11 +28,12 @@
       <visual>
         <geometry>
-          <box size="0.2 0.4 0.7" />
+          <box size="0.16 0.32 0.56" />
         </geometry>
         <material name="dark_grey" />
       </visual>
       <collision>
-        <geometry>
-          <box size="0.2 0.4 0.6" />
+        <origin xyz="0 0 -0.25" />
+        <geometry>
+          <cylinder length="1.5" radius="0.3" />
         </geometry>
       </collision>
@@ -39,5 +41,5 @@
     <!-- depth perception lidar -->
     <joint name="lidar_joint" type="fixed">
-      <origin xyz="0.15 0 0" rpy="0 0 0" />
+      <origin xyz="0.3 0 0" rpy="0 0 0" />
       <parent link="base_link"/>
       <child link="lidar_link" />
@@ -54,5 +56,5 @@
     <!-- left leg -->
     <joint name="left_leg_joint" type="fixed">
-      <origin xyz="0.0 0.11 -0.35" rpy="0 0 0" />
+      <origin xyz="0.0 0.09 -0.28" rpy="0 0 0" />
       <parent link="base_link"/>
       <child link="left_leg_link" />
@@ -60,27 +62,22 @@
     <link name="left_leg_link">
       <inertial>
-        <mass value="40" />
-        <origin xyz="0 0 0" />
-        <inertia ixx="1.0" ixy="0.0" ixz="0.0"
-          iyy="1.0" iyz="0.0"
-          izz="1.0" />
-      </inertial>
-      <visual>
-        <origin xyz="0 0 -0.45" />
-        <geometry>
-          <cylinder length="0.9" radius="0.09" />
-        </geometry>
-        <material name="dark_grey" />
-      </visual>
-      <collision>
-        <origin xyz="0 0 -0.45" />
-        <geometry>
-          <cylinder length="0.9" radius="0.09" />
-        </geometry>
-      </collision>
-    </link>
+        <mass value="0.01" />
+        <origin xyz="0 0 0" />
+        <inertia ixx="0.001" ixy="0.0" ixz="0.0"
+          iyy="0.001" iyz="0.0"
+          izz="0.001" />
+      </inertial>
+      <visual>
+        <origin xyz="0 0 -0.36" />
+        <geometry>
+          <cylinder length="0.72" radius="0.07" />
+        </geometry>
+        <material name="dark_grey" />
+      </visual>
+    </link>
+    <xacro:default_surface name="left_leg" />
     <!-- right leg -->
     <joint name="right_leg_joint" type="fixed">
-      <origin xyz="0.0 -0.11 -0.35" rpy="0 0 0" />
+      <origin xyz="0.0 -0.09 -0.28" rpy="0 0 0" />
       <parent link="base_link"/>
       <child link="right_leg_link" />
@@ -88,27 +85,22 @@
     <link name="right_leg_link">
       <inertial>
-        <mass value="40" />
-        <origin xyz="0 0 0" />
-        <inertia ixx="1.0" ixy="0.0" ixz="0.0"
-          iyy="1.0" iyz="0.0"
-          izz="1.0" />
-      </inertial>
-      <visual>
-        <origin xyz="0 0 -0.45" />
-        <geometry>
-          <cylinder length="0.9" radius="0.09" />
-        </geometry>
-        <material name="dark_grey" />
-      </visual>
-      <collision>
-        <origin xyz="0 0 -0.45" />
-        <geometry>
-          <cylinder length="0.9" radius="0.09" />
-        </geometry>
-      </collision>
-    </link>
+        <mass value="0.01" />
+        <origin xyz="0 0 0" />
+        <inertia ixx="0.001" ixy="0.0" ixz="0.0"
+          iyy="0.001" iyz="0.0"
+          izz="0.001" />
+      </inertial>
+      <visual>
+        <origin xyz="0 0 -0.36" />
+        <geometry>
+          <cylinder length="0.72" radius="0.07" />
+        </geometry>
+        <material name="dark_grey" />
+      </visual>
+    </link>
+    <xacro:default_surface name="right_leg" />
     <!-- head -->
     <joint name="head_joint" type="fixed">
-      <origin xyz="0 0 0.5" rpy="0 0 0" />
+      <origin xyz="0 0 0.43" rpy="0 0 0" />
       <parent link="base_link"/>
       <child link="head_link" />
@@ -116,9 +108,9 @@
     <link name="head_link">
       <inertial>
-        <mass value="20" />
-        <origin xyz="0 0 0" />
-        <inertia ixx="1.0" ixy="0.0" ixz="0.0"
-          iyy="1.0" iyz="0.0"
-          izz="1.0" />
+        <mass value="0.01" />
+        <origin xyz="0 0 0" />
+        <inertia ixx="0.001" ixy="0.0" ixz="0.0"
+          iyy="0.001" iyz="0.0"
+          izz="0.001" />
       </inertial>
       <visual>
@@ -128,9 +120,4 @@
         <material name="dark_grey" />
       </visual>
-      <collision>
-        <geometry>
-          <sphere radius="0.15" />
-        </geometry>
-      </collision>
     </link>
     <!-- camera -->
@@ -144,7 +131,7 @@
         <mass value="0.001" />
         <origin xyz="0 0 0" />
-        <inertia ixx="0.01" ixy="0.0" ixz="0.0"
-          iyy="0.01" iyz="0.0"
-          izz="0.01" />
+        <inertia ixx="0.001" ixy="0.0" ixz="0.0"
+          iyy="0.001" iyz="0.0"
+          izz="0.001" />
       </inertial>
     </link>
@@ -159,12 +146,12 @@
         <mass value="0.001" />
         <origin xyz="0 0 0" />
-        <inertia ixx="0.01" ixy="0.0" ixz="0.0"
-          iyy="0.01" iyz="0.0"
-          izz="0.01" />
+        <inertia ixx="0.001" ixy="0.0" ixz="0.0"
+          iyy="0.001" iyz="0.0"
+          izz="0.001" />
       </inertial>
     </link>
     <!-- left arm -->
     <joint name="left_arm_joint" type="fixed">
-      <origin xyz="0 0.27 0.28" rpy="0 ${M_PI} 0" />
+      <origin xyz="0 0.22 0.22" rpy="0 ${M_PI} 0" />
       <parent link="base_link"/>
       <child link="left_arm_link" />
@@ -172,27 +159,21 @@
     <link name="left_arm_link">
       <inertial>
-        <mass value="20" />
-        <origin xyz="0 0 0" />
-        <inertia ixx="1.0" ixy="0.0" ixz="0.0"
-          iyy="1.0" iyz="0.0"
-          izz="1.0" />
-      </inertial>
-      <visual>
-        <origin xyz="0 0 0.175" />
-        <geometry>
-          <cylinder length="0.35" radius="0.07" />
-        </geometry>
-        <material name="dark_grey" />
-      </visual>
-      <collision>
-        <origin xyz="0 0 0.175" />
-        <geometry>
-          <cylinder length="0.35" radius="0.07" />
-        </geometry>
-      </collision>
+        <mass value="0.01" />
+        <origin xyz="0 0 0" />
+        <inertia ixx="0.001" ixy="0.0" ixz="0.0"
+          iyy="0.001" iyz="0.0"
+          izz="0.001" />
+      </inertial>
+      <visual>
+        <origin xyz="0 0 0.14" />
+        <geometry>
+          <cylinder length="0.28" radius="0.06" />
+        </geometry>
+        <material name="dark_grey" />
+      </visual>
     </link>
     <!-- left fore arm -->
     <joint name="left_forearm_joint" type="fixed">
-      <origin xyz="0 0 0.35" rpy="0 -${M_PI/6} 0" />
+      <origin xyz="0 0 0.28" rpy="0 -${M_PI/6} 0" />
       <parent link="left_arm_link"/>
       <child link="left_forearm_link" />
@@ -200,27 +181,21 @@
     <link name="left_forearm_link">
       <inertial>
-        <mass value="20" />
-        <origin xyz="0 0 0" />
-        <inertia ixx="1.0" ixy="0.0" ixz="0.0"
-          iyy="1.0" iyz="0.0"
-          izz="1.0" />
-      </inertial>
-      <visual>
-        <origin xyz="0 0 0.175" />
-        <geometry>
-          <cylinder length="0.35" radius="0.07" />
-        </geometry>
-        <material name="dark_grey" />
-      </visual>
-      <collision>
-        <origin xyz="0 0 0.175" />
-        <geometry>
-          <cylinder length="0.35" radius="0.07" />
-        </geometry>
-      </collision>
+        <mass value="0.01" />
+        <origin xyz="0 0 0" />
+        <inertia ixx="0.001" ixy="0.0" ixz="0.0"
+          iyy="0.001" iyz="0.0"
+          izz="0.001" />
+      </inertial>
+      <visual>
+        <origin xyz="0 0 0.14" />
+        <geometry>
+          <cylinder length="0.28" radius="0.06" />
+        </geometry>
+        <material name="dark_grey" />
+      </visual>
     </link>
     <!-- right arm -->
     <joint name="right_arm_joint" type="fixed">
-      <origin xyz="0 -0.27 0.28" rpy="0 ${M_PI} 0" />
+      <origin xyz="0 -0.22 0.22" rpy="0 ${M_PI} 0" />
       <parent link="base_link"/>
       <child link="right_arm_link" />
@@ -228,27 +203,21 @@
     <link name="right_arm_link">
       <inertial>
-        <mass value="20" />
-        <origin xyz="0 0 0" />
-        <inertia ixx="1.0" ixy="0.0" ixz="0.0"
-          iyy="1.0" iyz="0.0"
-          izz="1.0" />
-      </inertial>
-      <visual>
-        <origin xyz="0 0 0.175" />
-        <geometry>
-          <cylinder length="0.35" radius="0.07" />
-        </geometry>
-        <material name="dark_grey" />
-      </visual>
-      <collision>
-        <origin xyz="0 0 0.175" />
-        <geometry>
-          <cylinder length="0.35" radius="0.07" />
-        </geometry>
-      </collision>
+        <mass value="0.01" />
+        <origin xyz="0 0 0" />
+        <inertia ixx="0.001" ixy="0.0" ixz="0.0"
+          iyy="0.001" iyz="0.0"
+          izz="0.001" />
+      </inertial>
+      <visual>
+        <origin xyz="0 0 0.14" />
+        <geometry>
+          <cylinder length="0.28" radius="0.06" />
+        </geometry>
+        <material name="dark_grey" />
+      </visual>
     </link>
     <!-- right fore arm -->
     <joint name="right_forearm_joint" type="fixed">
-      <origin xyz="0 0 0.35" rpy="0 -${M_PI/6} 0" />
+      <origin xyz="0 0 0.28" rpy="0 -${M_PI/6} 0" />
       <parent link="right_arm_link"/>
       <child link="right_forearm_link" />
@@ -256,30 +225,22 @@
     <link name="right_forearm_link">
       <inertial>
-        <mass value="20" />
-        <origin xyz="0 0 0" />
-        <inertia ixx="1.0" ixy="0.0" ixz="0.0"
-          iyy="1.0" iyz="0.0"
-          izz="1.0" />
-      </inertial>
-      <visual>
-        <origin xyz="0 0 0.175" />
-        <geometry>
-          <cylinder length="0.35" radius="0.07" />
-        </geometry>
-        <material name="dark_grey" />
-      </visual>
-      <collision>
-        <origin xyz="0 0 0.175" />
-        <geometry>
-          <cylinder length="0.35" radius="0.07" />
-        </geometry>
-      </collision>
-    </link>
-  <!-- <gazebo> -->
-  <!--   <canonicalBody>base_footprint</canonicalBody> -->
-  <!--   <controller:personcontroller_plugin name="controller" plugin="libpersoncontroller_plugin.so"> -->
-  <!--     <topicName>cmd_vel</topicName> -->
-  <!--   </controller:personcontroller_plugin> -->
-  <!-- </gazebo> -->
+        <mass value="0.01" />
+        <origin xyz="0 0 0" />
+        <inertia ixx="0.001" ixy="0.0" ixz="0.0"
+          iyy="0.001" iyz="0.0"
+          izz="0.001" />
+      </inertial>
+      <visual>
+        <origin xyz="0 0 0.14" />
+        <geometry>
+          <cylinder length="0.28" radius="0.06" />
+        </geometry>
+        <material name="dark_grey" />
+      </visual>
+    </link>
+    <gazebo>
+      <xacro:gazebo_person_drive />
+      <xacro:gazebo_ros_controller />
+    </gazebo>
   </xacro:macro>
 </root>
