Commit message: getting the camera to work - almost there. seems to be pointing weirdly. works with current setup if I use optical link, but the orientation is not right

File: bwi_gazebo_entities/gazebo/controllable_person.gazebo.xacro (robot description, xacro)
@@ -6,5 +6,5 @@
   <xacro:macro name="generic_camera" params="name">
     <gazebo reference="${name}_link">
-      <sensor:camera name="${name}_link_sensor">
+      <sensor:camera name="${name}_sensor">
         <imageFormat>R8G8B8</imageFormat>
         <imageSize>640 480</imageSize>
@@ -13,5 +13,5 @@
         <farClip>5</farClip>
         <updateRate>20.0</updateRate>
-        <controller:gazebo_ros_camera name="${name}_frame_controller" plugin="libgazebo_ros_camera.so">
+        <controller:gazebo_ros_camera name="${name}_controller" plugin="libgazebo_ros_prosilica.so">
           <alwaysOn>true</alwaysOn>
           <updateRate>20.0</updateRate>
@@ -25,5 +25,6 @@
           <distortionT1>0.00000001</distortionT1>
           <distortionT2>0.00000001</distortionT2>
-        </controller:gazebo_ros_openni_kinect>
+          <interface:camera name="${name}_iface"/>
+        </controller:gazebo_ros_camera>
       </sensor:camera>
     </gazebo>

File: bwi_gazebo_entities/urdf/person.urdf.xacro (robot description, xacro)
@@ -123,5 +123,5 @@
     <!-- camera -->
     <joint name="camera_joint" type="fixed">
-      <origin xyz="0.15 0 0" rpy="0 0 0" />
+      <origin xyz="0.16 0 0" rpy="0 0 0" />
       <parent link="head_link"/>
       <child link="camera_link" />

Commit message: a number of small improvements to the test environment

File: bwi_gazebo_entities/gazebo/controllable_person.gazebo.xacro (robot description, xacro)
@@ -10,6 +10,6 @@
         <imageSize>640 480</imageSize>
         <hfov>60</hfov>
-        <nearClip>0.01</nearClip>
-        <farClip>20</farClip>
+        <nearClip>0.1</nearClip>
+        <farClip>30</farClip>
         <updateRate>20.0</updateRate>
         <controller:gazebo_ros_camera name="${name}_controller" plugin="libgazebo_ros_prosilica.so">

File: bwi_gazebo_entities/urdf/person.urdf.xacro (robot description, xacro)
@@ -13,5 +13,5 @@
     </link>
     <joint name="base_link_joint" type="fixed">
-      <origin xyz="0.0 0 1.0" rpy="0 0 0" />
+      <origin xyz="0.0 0 1.25" rpy="0 0 0" />
       <parent link="base_footprint"/>
       <child link="base_link" />
@@ -28,12 +28,12 @@
       <visual>
         <geometry>
-          <box size="0.16 0.32 0.56" />
+          <box size="0.2 0.4 0.7" />
         </geometry>
         <material name="dark_grey" />
       </visual>
       <collision>
-        <origin xyz="0 0 -0.25" />
-        <geometry>
-          <cylinder length="1.5" radius="0.05" />
+        <origin xyz="0 0 -0.35" />
+        <geometry>
+          <cylinder length="1.8" radius="0.05" />
         </geometry>
       </collision>
@@ -56,5 +56,5 @@
     <!-- left leg -->
     <joint name="left_leg_joint" type="fixed">
-      <origin xyz="0.0 0.09 -0.28" rpy="0 0 0" />
+      <origin xyz="0.0 0.11 -0.35" rpy="0 0 0" />
       <parent link="base_link"/>
       <child link="left_leg_link" />
@@ -69,7 +69,7 @@
       </inertial>
       <visual>
-        <origin xyz="0 0 -0.36" />
-        <geometry>
-          <cylinder length="0.72" radius="0.07" />
+        <origin xyz="0 0 -0.45" />
+        <geometry>
+          <cylinder length="0.9" radius="0.09" />
         </geometry>
         <material name="dark_grey" />
@@ -79,5 +79,5 @@
     <!-- right leg -->
     <joint name="right_leg_joint" type="fixed">
-      <origin xyz="0.0 -0.09 -0.28" rpy="0 0 0" />
+      <origin xyz="0.0 -0.11 -0.35" rpy="0 0 0" />
       <parent link="base_link"/>
       <child link="right_leg_link" />
@@ -92,7 +92,7 @@
       </inertial>
       <visual>
-        <origin xyz="0 0 -0.36" />
-        <geometry>
-          <cylinder length="0.72" radius="0.07" />
+        <origin xyz="0 0 -0.45" />
+        <geometry>
+          <cylinder length="0.9" radius="0.09" />
         </geometry>
         <material name="dark_grey" />
@@ -102,5 +102,5 @@
     <!-- head -->
     <joint name="head_joint" type="fixed">
-      <origin xyz="0 0 0.43" rpy="0 0 0" />
+      <origin xyz="0 0 0.50" rpy="0 0 0" />
       <parent link="base_link"/>
       <child link="head_link" />
@@ -123,5 +123,5 @@
     <!-- camera -->
     <joint name="camera_joint" type="fixed">
-      <origin xyz="-1.0 0 0.5" rpy="0 ${M_PI/6} 0" />
+      <origin xyz="-1.0 0 0.25" rpy="0 ${M_PI/12} 0" />
       <parent link="head_link"/>
       <child link="camera_link" />
@@ -153,5 +153,5 @@
     <!-- left arm -->
     <joint name="left_arm_joint" type="fixed">
-      <origin xyz="0 0.22 0.22" rpy="0 ${M_PI} 0" />
+      <origin xyz="0 0.27 0.28" rpy="0 ${M_PI} 0" />
       <parent link="base_link"/>
       <child link="left_arm_link" />
@@ -166,7 +166,7 @@
       </inertial>
       <visual>
-        <origin xyz="0 0 0.14" />
-        <geometry>
-          <cylinder length="0.28" radius="0.06" />
+        <origin xyz="0 0 0.175" />
+        <geometry>
+          <cylinder length="0.35" radius="0.07" />
         </geometry>
         <material name="dark_grey" />
@@ -175,5 +175,5 @@
     <!-- left fore arm -->
     <joint name="left_forearm_joint" type="fixed">
-      <origin xyz="0 0 0.28" rpy="0 -${M_PI/6} 0" />
+      <origin xyz="0 0 0.35" rpy="0 -${M_PI/6} 0" />
       <parent link="left_arm_link"/>
       <child link="left_forearm_link" />
@@ -188,7 +188,7 @@
       </inertial>
       <visual>
-        <origin xyz="0 0 0.14" />
-        <geometry>
-          <cylinder length="0.28" radius="0.06" />
+        <origin xyz="0 0 0.175" />
+        <geometry>
+          <cylinder length="0.35" radius="0.07" />
         </geometry>
         <material name="dark_grey" />
@@ -197,5 +197,5 @@
     <!-- right arm -->
     <joint name="right_arm_joint" type="fixed">
-      <origin xyz="0 -0.22 0.22" rpy="0 ${M_PI} 0" />
+      <origin xyz="0 -0.27 0.28" rpy="0 ${M_PI} 0" />
       <parent link="base_link"/>
       <child link="right_arm_link" />
@@ -210,7 +210,7 @@
       </inertial>
       <visual>
-        <origin xyz="0 0 0.14" />
-        <geometry>
-          <cylinder length="0.28" radius="0.06" />
+        <origin xyz="0 0 0.175" />
+        <geometry>
+          <cylinder length="0.35" radius="0.07" />
         </geometry>
         <material name="dark_grey" />
@@ -219,5 +219,5 @@
     <!-- right fore arm -->
     <joint name="right_forearm_joint" type="fixed">
-      <origin xyz="0 0 0.28" rpy="0 -${M_PI/6} 0" />
+      <origin xyz="0 0 0.35" rpy="0 -${M_PI/6} 0" />
       <parent link="right_arm_link"/>
       <child link="right_forearm_link" />
@@ -232,7 +232,7 @@
       </inertial>
       <visual>
-        <origin xyz="0 0 0.14" />
-        <geometry>
-          <cylinder length="0.28" radius="0.06" />
+        <origin xyz="0 0 0.175" />
+        <geometry>
+          <cylinder length="0.35" radius="0.07" />
         </geometry>
         <material name="dark_grey" />
