Commit message: changing the person model + fixes

File: bwi_gazebo_entities/urdf/person.gazebo.xacro (robot description, xacro)
@@ -27,6 +27,6 @@
       <topicName>cmd_vel</topicName>
       <mapTopic>map</mapTopic>
-      <modelRadius>0.3</modelRadius>
-      <robotPadding>0.025</robotPadding>
+      <modelRadius>0.2</modelRadius>
+      <modelPadding>0.025</modelPadding>
     </controller:person_drive_plugin>
   </xacro:macro>

File: bwi_gazebo_entities/urdf/person.urdf.xacro (robot description, xacro)
@@ -35,5 +35,5 @@
         <origin xyz="0 0 -0.25" />
         <geometry>
-          <cylinder length="1.5" radius="0.3" />
+          <cylinder length="1.5" radius="0.2" />
         </geometry>
       </collision>
@@ -123,5 +123,5 @@
     <!-- camera -->
     <joint name="camera_joint" type="fixed">
-      <origin xyz="0.16 0 0" rpy="0 0 0" />
+      <origin xyz="-1.0 0 0.5" rpy="0 ${M_PI/6} 0" />
       <parent link="head_link"/>
       <child link="camera_link" />
@@ -241,5 +241,5 @@
     <gazebo>
       <xacro:gazebo_person_drive />
-      <xacro:gazebo_ros_controller />
+      <!-- <xacro:gazebo_ros_controller_manager /> -->
     </gazebo>
   </xacro:macro>
