Commit message: added a red ball model as the goal of the experiment

File: bwi_gazebo_entities/urdf/common.urdf.xacro (robot description, xacro)
@@ -10,3 +10,6 @@
     <color rgba="0.4 0.4 0.4 1" />
   </material>
+  <material name="red">
+    <color rgba="1.0 0.0 0.0 1" />
+  </material>
 </root>
