Commit message: removed teleport in favor of gazebo set model state, introduced pause feature in gazebo plugin, made teleport more robust, removed object controller plugin from robots and ball, added secondary experiment for testing

File: bwi_gazebo_entities/urdf/ball.urdf.xacro (robot description, xacro)
@@ -13,5 +13,5 @@
     </link>
     <joint name="base_link_joint" type="fixed">
-      <origin xyz="0.0 0 0.5" rpy="0 0 0" />
+      <origin xyz="0.0 0 0.3" rpy="0 0 0" />
       <parent link="base_footprint"/>
       <child link="base_link" />
@@ -28,5 +28,5 @@
       <visual>
         <geometry>
-          <sphere radius="0.5" />
+          <sphere radius="0.3" />
         </geometry>
         <material name="red" />
@@ -34,5 +34,5 @@
       <collision>
         <geometry>
-          <sphere radius="0.5" />
+          <sphere radius="0.3" />
         </geometry>
       </collision>
@@ -41,7 +41,4 @@
       <material>Gazebo/Red</material>
     </gazebo>
-    <gazebo>
-      <xacro:gazebo_person_drive />
-    </gazebo>
   </xacro:macro>
 </root>

Commit message: marginally increased the size of the goal ball

File: bwi_gazebo_entities/urdf/ball.urdf.xacro (robot description, xacro)
@@ -13,5 +13,5 @@
     </link>
     <joint name="base_link_joint" type="fixed">
-      <origin xyz="0.0 0 0.3" rpy="0 0 0" />
+      <origin xyz="0.0 0 0.4" rpy="0 0 0" />
       <parent link="base_footprint"/>
       <child link="base_link" />
@@ -28,5 +28,5 @@
       <visual>
         <geometry>
-          <sphere radius="0.3" />
+          <sphere radius="0.4" />
         </geometry>
         <material name="red" />
@@ -34,5 +34,5 @@
       <collision>
         <geometry>
-          <sphere radius="0.3" />
+          <sphere radius="0.4" />
         </geometry>
       </collision>
