Commit message: reduced the size of the robot model, and increased mass. It is now much easier to navigate around robots

File: bwi_gazebo_entities/urdf/person.urdf.xacro (robot description, xacro)
@@ -20,5 +20,5 @@
     <link name="base_link">
       <inertial>
-        <mass value="0.01" />
+        <mass value="50" />
         <origin xyz="0 0 0" />
         <inertia ixx="1.0" ixy="0.0" ixz="0.0"
@@ -35,5 +35,5 @@
         <origin xyz="0 0 -0.25" />
         <geometry>
-          <cylinder length="1.5" radius="0.15" />
+          <cylinder length="1.5" radius="0.05" />
         </geometry>
       </collision>
@@ -62,9 +62,9 @@
     <link name="left_leg_link">
       <inertial>
-        <mass value="0.01" />
-        <origin xyz="0 0 0" />
-        <inertia ixx="0.001" ixy="0.0" ixz="0.0"
-          iyy="0.001" iyz="0.0"
-          izz="0.001" />
+        <mass value="50" />
+        <origin xyz="0 0 0" />
+        <inertia ixx="1.0" ixy="0.0" ixz="0.0"
+          iyy="1.0" iyz="0.0"
+          izz="1.0" />
       </inertial>
       <visual>
@@ -85,9 +85,9 @@
     <link name="right_leg_link">
       <inertial>
-        <mass value="0.01" />
-        <origin xyz="0 0 0" />
-        <inertia ixx="0.001" ixy="0.0" ixz="0.0"
-          iyy="0.001" iyz="0.0"
-          izz="0.001" />
+        <mass value="50" />
+        <origin xyz="0 0 0" />
+        <inertia ixx="1.0" ixy="0.0" ixz="0.0"
+          iyy="1.0" iyz="0.0"
+          izz="1.0" />
       </inertial>
       <visual>

Commit message: messing around with the person model to get a much simple model controller plugin to work

File: bwi_gazebo_entities/urdf/person.urdf.xacro (robot description, xacro)
@@ -21,8 +21,8 @@
       <inertial>
         <mass value="50" />
-        <origin xyz="0 0 0" />
-        <inertia ixx="1.0" ixy="0.0" ixz="0.0"
-          iyy="1.0" iyz="0.0"
-          izz="1.0" />
+        <origin xyz="0 0 -1.25" />
+        <inertia ixx="50.0" ixy="0.0" ixz="0.0"
+          iyy="50.0" iyz="0.0"
+          izz="50.0" />
       </inertial>
       <visual>
@@ -30,10 +30,9 @@
           <box size="0.2 0.4 0.7" />
         </geometry>
-        <material name="dark_grey" />
       </visual>
       <collision>
-        <origin xyz="0 0 -0.35" />
-        <geometry>
-          <cylinder length="1.8" radius="0.05" />
+        <origin xyz="0 0 -1.0" />
+        <geometry>
+          <cylinder length="0.5" radius="0.25" />
         </geometry>
       </collision>
@@ -62,5 +61,5 @@
     <link name="left_leg_link">
       <inertial>
-        <mass value="50" />
+        <mass value="0.001" />
         <origin xyz="0 0 0" />
         <inertia ixx="1.0" ixy="0.0" ixz="0.0"
@@ -85,5 +84,5 @@
     <link name="right_leg_link">
       <inertial>
-        <mass value="50" />
+        <mass value="0.001" />
         <origin xyz="0 0 0" />
         <inertia ixx="1.0" ixy="0.0" ixz="0.0"
@@ -108,5 +107,5 @@
     <link name="head_link">
       <inertial>
-        <mass value="0.01" />
+        <mass value="0.001" />
         <origin xyz="0 0 0" />
         <inertia ixx="0.001" ixy="0.0" ixz="0.0"
@@ -159,5 +158,5 @@
     <link name="left_arm_link">
       <inertial>
-        <mass value="0.01" />
+        <mass value="0.001" />
         <origin xyz="0 0 0" />
         <inertia ixx="0.001" ixy="0.0" ixz="0.0"
@@ -181,5 +180,5 @@
     <link name="left_forearm_link">
       <inertial>
-        <mass value="0.01" />
+        <mass value="0.001" />
         <origin xyz="0 0 0" />
         <inertia ixx="0.001" ixy="0.0" ixz="0.0"
@@ -203,5 +202,5 @@
     <link name="right_arm_link">
       <inertial>
-        <mass value="0.01" />
+        <mass value="0.001" />
         <origin xyz="0 0 0" />
         <inertia ixx="0.001" ixy="0.0" ixz="0.0"
@@ -225,5 +224,5 @@
     <link name="right_forearm_link">
       <inertial>
-        <mass value="0.01" />
+        <mass value="0.001" />
         <origin xyz="0 0 0" />
         <inertia ixx="0.001" ixy="0.0" ixz="0.0"

Commit message: created a small experiment with 2-3 instances of reaching goal idx 33

File: bwi_gazebo_entities/urdf/person.urdf.xacro (robot description, xacro)
@@ -122,8 +122,13 @@
     <!-- camera -->
     <joint name="camera_joint" type="fixed">
-      <origin xyz="-1.0 0 0.25" rpy="0 ${M_PI/12} 0" />
+      <origin xyz="0.151 0 0" rpy="0 ${M_PI/12} 0" />
       <parent link="head_link"/>
       <child link="camera_link" />
     </joint>
+    <!-- <joint name="camera_joint" type="fixed"> -->
+    <!--   <origin xyz="-1.0 0 0.25" rpy="0 ${M_PI/12} 0" /> -->
+    <!--   <parent link="head_link"/> -->
+    <!--   <child link="camera_link" /> -->
+    <!-- </joint> -->
     <link name="camera_link">
       <inertial>
