Commit message: updated urdf files - now control a lot better

File: bwi_gazebo_entities/persons/controllable_person.urdf (robot description, URDF)
Before this commit: robot person, 12 links, 11 joints
Links:
- link base_link: geometry collision cylinder length=1.5 radius=0.15; visual box size=0.16 0.32 0.56
Joints:
- joint camera_joint: origin xyz=-2.0 0 0.5 rpy=0 0.523598775598 0 -> xyz=-1.0 0 0.5 rpy=0 0.523598775598 0

File: bwi_gazebo_entities/urdf/person.gazebo.xacro (robot description, xacro)
@@ -27,5 +27,5 @@
       <topicName>cmd_vel</topicName>
       <mapTopic>map</mapTopic>
-      <modelRadius>0.2</modelRadius>
+      <modelRadius>0.15</modelRadius>
       <modelPadding>0.025</modelPadding>
     </controller:person_drive_plugin>

File: bwi_gazebo_entities/urdf/person.urdf.xacro (robot description, xacro)
@@ -35,5 +35,5 @@
         <origin xyz="0 0 -0.25" />
         <geometry>
-          <cylinder length="1.5" radius="0.2" />
+          <cylinder length="1.5" radius="0.15" />
         </geometry>
       </collision>
